File: sensor9dof.brd (EAGLE design)
At the start: 100 x 100 mm, 12 parts, among them IC1 BMI160, IC2 BMM150, X1 TSW-114-02-S-S, X2 TSW-114-02-S-S

Commit message: r0.1
Parts:
- ICON2: value (none) -> r0.1
Changed lines of the file:
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@@
 <attribute name="NOT_COMPONENT" value="YES" x="20.1" y="8.1" size="1.7" layer="27" ratio="18" display="off"/>
 </element>
-<element name="ICON2" library="mylib" package="ICON_REVISION2.0" value="" x="26.4" y="7.3">
+<element name="ICON2" library="mylib" package="ICON_REVISION2.0" value="r0.1" x="26.4" y="7.3">
 <attribute name="NOT_COMPONENT" value="YES" x="26.4" y="7.3" size="1.7" layer="27" ratio="18" display="off"/>
 </element>
