File: sensor9dof.sch (EAGLE design)
At the start: 12 parts, among them IC1 BMI160, IC2 BMM150, X1 TSW-114-02-S-S, X2 TSW-114-02-S-S

Commit message: r0.1
Parts:
- ICON2: value (none) -> r0.1
Changed lines of the file:
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@@
 <part name="X1" library="mylib" deviceset="TSW-114-02-S-S" device=""/>
 <part name="ICON1" library="mylib" deviceset="ICON_OSHW" device=""/>
-<part name="ICON2" library="mylib" deviceset="ICON_REVISION" device="_2.0"/>
+<part name="ICON2" library="mylib" deviceset="ICON_REVISION" device="_2.0" value="r0.1"/>
 <part name="P5" library="mylib" deviceset="PCB_CORNER" device="_NH"/>
 <part name="P6" library="mylib" deviceset="PCB_CORNER" device=""/>
@@
 <instance part="X1" gate="-13" x="55.88" y="165.1" rot="MR180"/>
 <instance part="X1" gate="-14" x="55.88" y="167.64" rot="MR180"/>
-<instance part="ICON1" gate="G$1" x="246.38" y="22.86"/>
+<instance part="ICON1" gate="G$1" x="246.38" y="21.59"/>
 <instance part="ICON2" gate="G$1" x="162.56" y="7.62"/>
 <instance part="P5" gate="G$1" x="144.78" y="10.16" rot="R270"/>
